Commit message: Fix robot model orientation and add RPLidar to main launch
URDF orientation fix (chassis was drawn backwards):
- chassis_joint: add rpy="0 0 pi" rotation, adjust x to chassis_length-wheel_offset_x
- caster_wheel_offset_x: 0.033 -> 0.207 (now measured from front in flipped chassis frame)
- lidar.xacro: origin x 0.200 -> 0.040 (40mm from front edge in flipped frame)
- robot.urdf.xacro: comment out face.xacro inclusion

RPLidar integration:
- launch_robot.launch.py: include rplidar.launch.py in main launch

Co-Authored-By: Claude Sonnet 4.6 <noreply@anthropic.com>

File: src/articubot_one/description/lidar.xacro (robot description, xacro)
@@ -4,5 +4,5 @@
         <parent link="chassis"/>
         <child link="laser_frame"/>
-        <origin xyz="0.200 0 0.116" rpy="0 0 0"/>
+        <origin xyz="0.040 0 0.116" rpy="0 0 0"/>
     </joint>
     <link name="laser_frame">

File: src/articubot_one/description/robot_core.xacro (robot description, xacro)
@@ -14,5 +14,5 @@
     <xacro:property name="caster_wheel_radius" value="0.01"/>
     <xacro:property name="caster_wheel_mass" value="0.01"/>
-    <xacro:property name="caster_wheel_offset_x" value="0.033"/>
+    <xacro:property name="caster_wheel_offset_x" value="0.207"/>
     <xacro:property name="caster_wheel_offset_z" value="${wheel_offset_z - wheel_radius + caster_wheel_radius}"/>
     <material name="white">
@@ -46,5 +46,5 @@
         <parent link="base_link"/>
         <child link="chassis"/>
-        <origin xyz="${-wheel_offset_x} 0 ${-wheel_offset_z}"/>
+        <origin xyz="${chassis_length - wheel_offset_x} 0 ${-wheel_offset_z}" rpy="0 0 ${pi}"/>
     </joint>
     <link name="chassis">
