Commit message: Add SLAM, BNO055 IMU, and robot_localization EKF
- SLAM with slam_toolbox: fixed mode→mapping, use_sim_time→false,
  max_laser_range→12.0, minimum_travel_distance/heading→0.2
- Saved map: maps/my_map.pgm + my_map.yaml (200x136 @ 0.05m/pix)
- BNO055: ros-humble-bno055 on I2C bus 1 at 0x28, config/bno055_params.yaml
- robot_localization EKF: fuses /diff_cont/odom + /imu/imu → /odom at 20Hz
- imu_link added to URDF at xyz="0.004 -0.018 0.055"
- Removed old /diff_cont/odom→/odom remap; EKF now owns /odom
- Updated CLAUDE.md (fix history #13, #14) and HARDWARE_MEMORY.md
- Added BNO055 datasheet to Hardware/

Co-Authored-By: Claude Sonnet 4.6 <noreply@anthropic.com>

File: src/articubot_one/description/robot_core.xacro (robot description, xacro)
@@ -121,4 +121,12 @@
         <material>Gazebo/Blue</material>
     </gazebo>
+    <!-- IMU LINK -->
+    <joint name="imu_joint" type="fixed">
+        <parent link="base_link"/>
+        <child link="imu_link"/>
+        <origin xyz="0.004 -0.018 0.055" rpy="0 0 0"/>
+    </joint>
+    <link name="imu_link">
+    </link>
     <!-- CASTER WHEEL LINK -->
     <joint name="caster_wheel_joint" type="fixed">
